File: MM_PCB/MicroMouse_v0.brd (EAGLE design)
At the start: 76 x 96 mm, 0 parts

Commit message: Have MM layout finally semi finalized
Parts:
- added U$1: STM32F405XXSTM32F405XX, stm32f:LQFP64
Connections:
- new net VBAT: U$1.1
- new net VCAP_1: U$1.31
- new net VCAP_2: U$1.47
- new net VDD1: U$1.19
- new net VDD2: U$1.32
- new net VDD3: U$1.48
- new net VDD4: U$1.64
- new net VDDA: U$1.13
- new net VSS1: U$1.18
- new net VSS2: U$1.63
- new net VSSA: U$1.12
Other:
- board size 76 x 96 mm -> 76 x 90 mm
- board text added: "CUT OUT"
